File: Adafruit PowerBoost 1000C Rev B.sch (EAGLE design)
At the start: 42 parts, among them CN1 USBA_FEMALE, CN4 MicroUSB, T1 MMUN2133LT1G, U1 TPS61090RSAR, U2 MCP73871

Commit message: Mod
connected Data lines of both USB-connectors
Parts:
- added R15, R18: DNP, rcl:R-EU_R0603-VISHAY
- C2: device microbuilder:CAP_CERAMIC0805-NOOUTLINE -> rcl:C-EUC0603-VISHAY
- C4: device microbuilder:CAP_CERAMIC0805_10MGAP -> rcl:C-EUC0603-VISHAY
- CHRG/LBO, DONE, LED1, LED2: device microbuilder:LED0805_NOOUTLINE -> microbuilder:LED0603_NOOUTLINE
- R1, R2: device microbuilder:RESISTOR_0805MP -> rcl:R-EU_R0603-VISHAY
- R10, R11, R12, R14, R16, R17, R20, R3, R4, R5, R6, R7, R8, R9, THERM: device microbuilder:RESISTOR0805_NOOUTLINE -> rcl:R-EU_R0603-VISHAY
Connections:
- net D+: now also CN4.D+, R18.1, R18.2
- net D-: now also CN4.D-, R15.1, R15.2
Other:
- moved on the sheet: C2, C4, JP2

Commit message: added PDF Schematic
Other:
- note added: "MOD"
- note added: "mod by tinyledmatrix"
